File: docs/assets/eagle/buscard.brd (EAGLE design)
At the start: 153.7 x 137.9 mm, 48 parts, among them P1 COMMODORE_64_EXPANSION_PORT_C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, P2 FEMALE_44-PIN_CARD_EDGE_CONNE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, P3 COMMODORE_IEEE-488_PORT_CARD_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, P4 Parallel Port, Q1 2N4401, Q2 2N3904, U1 TMS 2564, U10 74LS139N, U11 74LS21N, U12 74LS04N, U13 TMS 2564, U14 TMS 2564, U15 TMS 2564, U2 8255AC-5, U3 75160AN, U4 75161AN, U5 74LS32N, U6 74LS04N, U7 74LS08N, U8 74LS00N, U9 74LS21N

Commit message: Clarified diagnostic header info
Parts:
- J2: device mystery_plug-MTA04-100:10X04MTA -> diagnostic-header-MTA04-100:10X04MTA
Connections:
- net MP4 renamed BC-ROM-INACTIVE
Changed lines of the file:
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@@
 <attribute name="VALUE" x="103.505" y="118.364" size="1.27" layer="27" rot="R180"/>
 </element>
-<element name="J2" library="mystery_plug-MTA04-100" package="10X04MTA" value="" x="107.315" y="105.41" smashed="yes" rot="R180">
+<element name="J2" library="diagnostic-header-MTA04-100" package="10X04MTA" value="" x="107.315" y="105.41" smashed="yes" rot="R180">
 <attribute name="NAME" x="101.3968" y="106.0704" size="1.27" layer="25" rot="R180"/>
 <attribute name="VALUE" x="112.395" y="109.855" size="1.27" layer="27" rot="R180"/>
@@
 <wire x1="126.111" y1="36.2077" x2="123.825" y2="34.29" width="0.254" layer="16"/>
 </signal>
-<signal name="MP4">
+<signal name="BC-ROM-INACTIVE">
 <contactref element="U6" pad="13"/>
 <contactref element="U7" pad="4"/>
