File: docs/assets/eagle/buscard.sch (EAGLE design)
At the start: 48 parts, among them P1 COMMODORE_64_EXPANSION_PORT_C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, P2 FEMALE_44-PIN_CARD_EDGE_CONNE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, P3 COMMODORE_IEEE-488_PORT_CARD_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, P4 Parallel Port, Q1 2N4401, Q2 2N3904, U1 TMS 2564, U10 74LS139N, U11 74LS21N, U12 74LS04N, U13 TMS 2564, U14 TMS 2564, U15 TMS 2564, U2 8255AC-5, U3 75160AN, U4 75161AN, U5 74LS32N, U6 74LS04N, U7 74LS08N, U8 74LS00N, U9 74LS21N

Commit message: Clarified diagnostic header info
Parts:
- J2: device mystery_plug-MTA04-100:MTA04-100 -> diagnostic-header-MTA04-100:MTA04-100
Connections:
- net MP4 renamed BC-ROM-INACTIVE
Other:
- note added: "1"
- note added: "A reverse-engineered IEEE-488 and parallel printer interface for Commodore 64, based on the original BusCard (R) by Batteries Included Ltd., Toronto, Canada. The original 1983 circuit board is labeled as Revision A. For more information, see https://github.com/pdbuchan/buscard"
- note added: "Diagnostic/Test Header J2 provides access to !HIRAM!, !LORAM!, and the BusCard ROM-inactive status signal (BC-ROM-INACTIVE) for testing and troubleshooting."
- note added: "J1 for use with Type A C64 only: 2-pin header for clip leads to C64 !HIRAM! and !LORAM! signals at R44 and R45, respectively. Pin 1 of J1 connects to R44 using red clip, pin 2 to R45 using black clip. See BusCard manual for details."
- note added: "September 2026"
- note removed: "0"
- note removed: "A reverse-engineered IEEE-488 and parallel printer interface for Commodore 64, based on the original BusCard (R) by Batteries Included Ltd., Toronto, Canada. The original 1983 circuit board is labeled as Revision A. For more information, see pdbuchan.com."
- note removed: "Diagnostic Jack"
- note removed: "For use with Type A C64 only: Jack for clip-leads to C64 !HIRAM! and !LORAM! bits at R44 and R45, respectively. Pin 1 of J1 connects to R44 using red clip, pin 2 to R45 using black clip. See BusCard manual for details."
- note removed: "July 2017"
Changed lines of the file:
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@@
 <setting verticaltext="up"/>
 </settings>
-<grid distance="0.025" unitdist="inch" unit="inch" style="lines" multiple="1" display="no" altdistance="0.01" altunitdist="inch" altunit="inch"/>
+<grid distance="0.1" unitdist="inch" unit="inch" style="lines" multiple="1" display="no" altdistance="0.01" altunitdist="inch" altunit="inch"/>
 <layers>
 <layer number="1" name="Top" color="4" fill="1" visible="no" active="no"/>
@@
 <part name="S1" library="dip-switch-DS08" deviceset="DS08" device="" value="DIP Switch"/>
 <part name="J1" library="clip-header-MTA02-100" deviceset="MTA02-100" device=""/>
-<part name="J2" library="mystery_plug-MTA04-100" deviceset="MTA04-100" device=""/>
+<part name="J2" library="diagnostic-header-MTA04-100" deviceset="MTA04-100" device=""/>
 <part name="P4" library="commodore-card-edges" deviceset="COMMODORE_PARALLEL_PORT_CARD_EDGE" device="" value="Parallel Port"/>
 <part name="P3" library="commodore-card-edges" deviceset="COMMODORE_IEEE-488_PORT_CARD_EDGE" device=""/>
@@
 <text x="296.8625" y="-273.05" size="1.778" layer="96">P. David Buchan</text>
 <text x="296.8625" y="-242.57" size="1.778" layer="96">BusCard for Commodore 64</text>
-<text x="387.35" y="-242.57" size="2.54" layer="96">0</text>
+<text x="387.35" y="-242.57" size="2.54" layer="96">1</text>
 <text x="296.8625" y="-262.89" size="1.778" layer="96">A reverse-engineered IEEE-488 and parallel printer interface
 for Commodore 64, based on the original BusCard (R)
 by Batteries Included Ltd., Toronto, Canada.
 The original 1983 circuit board is labeled as Revision A.
-For more information, see pdbuchan.com.</text>
+For more information, see https://github.com/pdbuchan/buscard</text>
 <text x="208.915" y="-123.19" size="1.27" layer="91" rot="R90">N/C</text>
-<text x="240.03" y="-125.73" size="1.778" layer="96" rot="R180">Diagnostic Jack</text>
+<text x="280.67" y="-133.35" size="1.778" layer="96" rot="R180">Diagnostic/Test Header J2 provides access to !HIRAM!,
+!LORAM!, and the BusCard ROM-inactive status signal
+(BC-ROM-INACTIVE) for testing and troubleshooting.</text>
 <text x="-32.385" y="-93.0275" size="1.778" layer="91">PA0</text>
 <text x="-32.385" y="-95.5675" size="1.778" layer="91">PA1</text>
@@
 <text x="-32.385" y="-108.2675" size="1.778" layer="91">PA6</text>
 <text x="-32.385" y="-110.8075" size="1.778" layer="91">PA7</text>
-<text x="347.98" y="-273.05" size="1.778" layer="96">July 2017</text>
+<text x="347.98" y="-273.05" size="1.778" layer="96">September 2026</text>
 <text x="-55.88" y="-123.825" size="3.81" layer="96">Switch Functions and Settings</text>
 <text x="-55.88" y="-152.4" size="1.778" layer="96">Switches 1 and 2: Device 4 (printer)
@@
 Devices 11 and up have no switches and are
 permanently allocated to the BusCard IEEE-488 port.</text>
-<text x="264.795" y="-130.81" size="1.778" layer="96">For use with Type A C64 only:
-Jack for clip-leads
+<text x="264.795" y="-130.81" size="1.778" layer="96">J1 for use with Type A C64 only:
+2-pin header for clip leads
 to C64 !HIRAM! and !LORAM!
-bits at R44 and R45,
+signals at R44 and R45,
 respectively. Pin 1 of J1
 connects to R44 using red clip,
@@
 </segment>
 </net>
-<net name="MP4" class="0">
+<net name="BC-ROM-INACTIVE" class="0">
 <segment>
 <wire x1="181.61" y1="-208.915" x2="189.23" y2="-208.915" width="0.1524" layer="91"/>
